Commit message: poczatki lab3

File: lab2/urdf/movable.urdf (robot description, URDF)
Before this commit: robot manipulator, 4 links, 3 joints
Links:
- link link_3: geometry visual mesh filename=package://lab2/hand.stl scale=0.001 0.001 0.002

File: lab2/urdf/show.urdf (robot description, URDF)
Before this commit: robot manipulator, 4 links, 3 joints
Links:
- link link_3: geometry visual mesh filename=package://lab2/hand.stl scale=0.001 0.001 0.002

Commit message: lab3

File: lab2/urdf/movable.urdf (robot description, URDF)
Before this commit: robot manipulator, 4 links, 3 joints
Joints:
- joint base_to_link1: limit lower=-1.57075 upper=1.57075 effort=1000.0 velocity=0.5 -> lower=-3.1415 upper=3.1415 effort=1000.0 velocity=0.5
- joint link1_to_link2: limit lower=-1.57075 upper=1.57075 effort=1000.0 velocity=0.5 -> lower=-3.1415 upper=3.1415 effort=1000.0 velocity=0.5
- joint link2_to_link3: limit lower=0 upper=0.2 effort=1000.0 velocity=0.5 -> lower=-0.5 upper=0.5 effort=1000.0 velocity=0.5
